File: PCB/KiCAD Project/Starkit.kicad_pcb (KiCad board)
At the start: 2 copper layers, 65 x 112.5 mm, 34 parts, among them J1 Screw_Terminal_01x02, J11 Conn_01x06_Pin, J2 Screw_Terminal_01x02, J3 Screw_Terminal_01x02, J4 Screw_Terminal_01x02, J5 Conn_01x02, J6 Conn_01x02, U4 ESP32-DEVKITC-32D, X1 Conn_01x03_Pin, X2 Conn_01x03_Pin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

Commit message: 23-06-2025
Routing:
- net /12: track 119.9 -> 121.7 mm

Commit message: 09-07-2025
Parts:
- removed the G*** at (174.4, 132.8)
- added G***: LOGO, Starchip:Cat, F.Cu at (174.4, 132.8)
Routing:
- net /12: track 121.7 -> 119.9 mm

Commit message: 05/10/2025
Parts:
- removed the G*** at (126.2, 132.0)
- removed the G*** at (174.4, 132.8)
- added G***: LOGO, Starchip:Cat2, F.Cu at (173.8, 131.5)
- added G***: LOGO, Starchip:Heart, F.Cu at (151.5, 130.5)
- added G***: LOGO, Starchip:Hack_Club2, F.Cu at (128.0, 131.8)
Connections:
- J11 pad 2: /LiDAR_DATA -> /SDA
- J11 pad 3: /LiDAR_CLOCK -> /SCL
- U3 pad 3: /IMU_CLOCK -> /SCL
- U3 pad 4: /IMU_DATA -> /SDA
- U4 pad J3-11: /LiDAR_CLOCK -> unconnected-(U4-IO17-PadJ3-11)
- U4 pad J3-12: /LiDAR_DATA -> unconnected-(U4-IO16-PadJ3-12)
- U4 pad J3-3: /IMU_CLOCK -> /SCL
- U4 pad J3-6: /IMU_DATA -> /SDA
Routing:
- net /LiDAR_DATA: track 90.9 -> 0.00 mm
- net /LiDAR_CLOCK: track 89.4 -> 0.00 mm
- net /SDA: track 0.00 -> 58.3 mm
- net /SCL: track 0.00 -> 58.1 mm
- net /IMU_DATA: track 34.3 -> 0.00 mm
- net /IMU_CLOCK: track 33.8 -> 0.00 mm
- net /ESC: track 37.2 -> 35.4 mm, vias 1 -> 0
Other:
- board text added: "Made with for Highway"
- board text removed: "Made with love for Highway"
