File: PCB/KiCAD Project/Starkit.kicad_sch (KiCad schematic)
At the start: 25 parts, among them J1 Screw_Terminal_01x02, J11 Conn_01x06_Pin, J2 Screw_Terminal_01x02, J3 Screw_Terminal_01x02, J4 Screw_Terminal_01x02, J5 Conn_01x02, J6 Conn_01x02, U4 ESP32-DEVKITC-32D, X1 Conn_01x03_Pin, X2 Conn_01x03_Pin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

Commit message: 05/10/2025
Connections:
- net IMU_CLOCK renamed SCL
- net SCL: now also J11.3 (Pin_3)
- net IMU_DATA renamed SDA
- net SDA: now also J11.2 (Pin_2)
- net LiDAR_CLOCK: no longer names the net of U4.J3-11 (IO17)
- net LiDAR_CLOCK: no longer J11.3 (Pin_3)
- net LiDAR_DATA: no longer names the net of U4.J3-12 (IO16)
- net LiDAR_DATA: no longer J11.2 (Pin_2)
Changed lines of the file:
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@@
 		)
 	)
-	(label "LiDAR_DATA"
+	(label "SDA"
 		(at 135.89 82.55 0)
 		(effects
@@
 		)
 	)
-	(label "IMU_DATA"
+	(label "SDA"
 		(at 146.05 39.37 0)
 		(effects
@@
 		)
 	)
-	(label "LiDAR_CLOCK"
-		(at 109.22 107.95 0)
-		(effects
-			(font
-				(size 1.27 1.27)
-			)
-			(justify left bottom)
-		)
-	)
-	(label "IMU_CLOCK"
+	(label "SCL"
 		(at 109.22 87.63 0)
 		(effects
@@
 	(label "LED_B"
 		(at 109.22 85.09 0)
-		(effects
-			(font
-				(size 1.27 1.27)
-			)
-			(justify left bottom)
-		)
-	)
-	(label "LiDAR_DATA"
-		(at 109.22 110.49 0)
 		(effects
 			(font
@@
 		)
 	)
-	(label "LiDAR_CLOCK"
+	(label "SCL"
 		(at 138.43 85.09 0)
 		(effects
@@
 		)
 	)
-	(label "IMU_CLOCK"
+	(label "SCL"
 		(at 130.81 44.45 180)
 		(effects
@@
 		)
 	)
-	(label "IMU_DATA"
+	(label "SDA"
 		(at 109.22 95.25 0)
 		(effects
